File: design.kicad_sch (KiCad schematic)
At the start: 0 parts

Commit message: play around
Parts:
- added J1: 490107670412, Snapeda:490107670412_WURTH_490107670412, symbol Snapeda:490107670412
- added U1, U3: CH340C, Package_SO:SOIC-16_3.9x9.9mm_P1.27mm, symbol Interface_USB:CH340C
- added U2: TS3USB30RSWR, Snapeda:TS3USB30RSWR_QFN40P140X180X55-10N, symbol Snapeda:TS3USB30RSWR
Changed lines of the file:
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@@
     (comment 4 "<<hash>>")
+  )
+  (symbol (lib_id "Snapeda:490107670412") (at 170.18 60.96 0) (unit 1)
+    (in_bom yes) (on_board yes) (fields_autoplaced)
+    (property "Reference" "J1" (id 0) (at 170.18 50.8 0))
+    (property "Value" "490107670412" (id 1) (at 170.18 53.34 0))
+    (property "Footprint" "Snapeda:490107670412_WURTH_490107670412" (id 2) (at 170.18 60.96 0)
+      (effects (font (size 1.27 1.27)) (justify bottom) hide)
+    )
+    (property "Datasheet" "" (id 3) (at 170.18 60.96 0)
+      (effects (font (size 1.27 1.27)) hide)
+    )
+    (property "MF" "Wurth Elektronik" (id 4) (at 170.18 60.96 0)
+      (effects (font (size 1.27 1.27)) (justify bottom) hide)
+    )
+    (property "MAXIMUM_PACKAGE_HEIGHT" "10.45 mm" (id 5) (at 170.18 60.96 0)
+      (effects (font (size 1.27 1.27)) (justify bottom) hide)
+    )
+    (property "Package" "None" (id 6) (at 170.18 60.96 0)
+      (effects (font (size 1.27 1.27)) (justify bottom) hide)
+    )
+    (property "Price" "None" (id 7) (at 170.18 60.96 0)
+      (effects (font (size 1.27 1.27)) (justify bottom) hide)
+    )
+    (property "Check_prices" "https://www.snapeda.com/parts/490107670412/Wurth+Elektronik/view-part/?ref=eda" (id 8) (at 170.18 60.96 0)
+      (effects (font (size 1.27 1.27)) (justify bottom) hide)
+    )
+    (property "STANDARD" "Manufacturer Recommendations" (id 9) (at 170.18 60.96 0)
+      (effects (font (size 1.27 1.27)) (justify bottom) hide)
+    )
+    (property "PARTREV" "002.003" (id 10) (at 170.18 60.96 0)
+      (effects (font (size 1.27 1.27)) (justify bottom) hide)
+    )
+    (property "SnapEDA_Link" "https://www.snapeda.com/parts/490107670412/Wurth+Elektronik/view-part/?ref=snap" (id 11) (at 170.18 60.96 0)
+      (effects (font (size 1.27 1.27)) (justify bottom) hide)
+    )
+    (property "MP" "490107670412" (id 12) (at 170.18 60.96 0)
+      (effects (font (size 1.27 1.27)) (justify bottom) hide)
+    )
+    (property "Purchase-URL" "https://www.snapeda.com/api/url_track_click_mouser/?unipart_id=5159898&manufacturer=Wurth Elektronik&part_name=490107670412&search_term=skedd" (id 13) (at 170.18 60.96 0)
+      (effects (font (size 1.27 1.27)) (justify bottom) hide)
+    )
+    (property "Description" "\n4 Position Ribbon Cable Connector Black IDC 28 AWG Through Hole, SKEDD\n" (id 14) (at 170.18 60.96 0)
+      (effects (font (size 1.27 1.27)) (justify bottom) hide)
+    )
+    (property "Availability" "In Stock" (id 15) (at 170.18 60.96 0)
+      (effects (font (size 1.27 1.27)) (justify bottom) hide)
+    )
+    (property "MANUFACTURER" "Wuerth Elektronik" (id 16) (at 170.18 60.96 0)
+      (effects (font (size 1.27 1.27)) (justify bottom) hide)
+    )
+    (pin "1")
+    (pin "2")
+    (pin "3")
+    (pin "4")
+  )
+  (symbol (lib_id "Snapeda:TS3USB30RSWR") (at 59.055 83.82 0) (unit 1)
+    (in_bom yes) (on_board yes) (fields_autoplaced)
+    (property "Reference" "U2" (id 0) (at 59.055 63.5 0))
+    (property "Value" "TS3USB30RSWR" (id 1) (at 59.055 66.04 0))
+    (property "Footprint" "Snapeda:TS3USB30RSWR_QFN40P140X180X55-10N" (id 2) (at 59.055 83.82 0)
+      (effects (font (size 1.27 1.27)) (justify bottom) hide)
+    )
+    (property "Datasheet" "" (id 3) (at 59.055 83.82 0)
+      (effects (font (size 1.27 1.27)) hide)
+    )
+    (property "MF" "Texas Instruments" (id 4) (at 59.055 83.82 0)
+      (effects (font (size 1.27 1.27)) (justify bottom) hide)
+    )
+    (property "Description" "\nHigh-speed USB 2.0 (480-Mbps) 1:2 multiplexer & demultiplexer switch with single enable\n" (id 5) (at 59.055 83.82 0)
+      (effects (font (size 1.27 1.27)) (justify bottom) hide)
+    )
+    (property "PACKAGE" "UQFN-10" (id 6) (at 59.055 83.82 0)
+      (effects (font (size 1.27 1.27)) (justify bottom) hide)
+    )
+    (property "MPN" "TS3USB30RSWR" (id 7) (at 59.055 83.82 0)
+      (effects (font (size 1.27 1.27)) (justify bottom) hide)
+    )
+    (property "Price" "None" (id 8) (at 59.055 83.82 0)
+      (effects (font (size 1.27 1.27)) (justify bottom) hide)
+    )
+    (property "Package" "UQFN-10 Texas Instruments" (id 9) (at 59.055 83.82 0)
+      (effects (font (size 1.27 1.27)) (justify bottom) hide)
+    )
+    (property "OC_FARNELL" "1755574" (id 10) (at 59.055 83.82 0)
+      (effects (font (size 1.27 1.27)) (justify bottom) hide)
+    )
+    (property "SnapEDA_Link" "https://www.snapeda.com/parts/TS3USB30RSWR/Texas+Instruments/view-part/?ref=snap" (id 11) (at 59.055 83.82 0)
+      (effects (font (size 1.27 1.27)) (justify bottom) hide)
+    )
+    (property "MP" "TS3USB30RSWR" (id 12) (at 59.055 83.82 0)
+      (effects (font (size 1.27 1.27)) (justify bottom) hide)
+    )
+    (property "Purchase-URL" "https://www.snapeda.com/api/url_track_click_mouser/?unipart_id=60717&manufacturer=Texas Instruments&part_name=TS3USB30RSWR&search_term=ts3usb30" (id 13) (at 59.055 83.82 0)
+      (effects (font (size 1.27 1.27)) (justify bottom) hide)
+    )
+    (property "SUPPLIER" "Texas Instruments" (id 14) (at 59.055 83.82 0)
+      (effects (font (size 1.27 1.27)) (justify bottom) hide)
+    )
+    (property "OC_NEWARK" "45P8339" (id 15) (at 59.055 83.82 0)
+      (effects (font (size 1.27 1.27)) (justify bottom) hide)
+    )
+    (property "Availability" "In Stock" (id 16) (at 59.055 83.82 0)
+      (effects (font (size 1.27 1.27)) (justify bottom) hide)
+    )
+    (property "Check_prices" "https://www.snapeda.com/parts/TS3USB30RSWR/Texas+Instruments/view-part/?ref=eda" (id 17) (at 59.055 83.82 0)
+      (effects (font (size 1.27 1.27)) (justify bottom) hide)
+    )
+    (pin "1")
+    (pin "10")
+    (pin "2")
+    (pin "3")
+    (pin "4")
+    (pin "5")
+    (pin "6")
+    (pin "7")
+    (pin "8")
+    (pin "9")
+  )
+  (symbol (lib_id "Interface_USB:CH340C") (at 106.045 115.57 0) (unit 1)
+    (in_bom yes) (on_board yes) (fields_autoplaced)
+    (property "Reference" "U3" (id 0) (at 108.0644 131.445 0)
+      (effects (font (size 1.27 1.27)) (justify left))
+    )
+    (property "Value" "CH340C" (id 1) (at 108.0644 133.985 0)
+      (effects (font (size 1.27 1.27)) (justify left))
+    )
+    (property "Footprint" "Package_SO:SOIC-16_3.9x9.9mm_P1.27mm" (id 2) (at 107.315 129.54 0)
+      (effects (font (size 1.27 1.27)) (justify left) hide)
+    )
+    (property "Datasheet" "https://datasheet.lcsc.com/szlcsc/Jiangsu-Qin-Heng-CH340C_C84681.pdf" (id 3) (at 97.155 95.25 0)
+      (effects (font (size 1.27 1.27)) hide)
+    )
+    (pin "1")
+    (pin "10")
+    (pin "11")
+    (pin "12")
+    (pin "13")
+    (pin "14")
+    (pin "15")
+    (pin "16")
+    (pin "2")
+    (pin "3")
+    (pin "4")
+    (pin "5")
+    (pin "6")
+    (pin "7")
+    (pin "8")
+    (pin "9")
+  )
+  (symbol (lib_id "Interface_USB:CH340C") (at 106.68 55.245 0) (unit 1)
+    (in_bom yes) (on_board yes) (fields_autoplaced)
+    (property "Reference" "U1" (id 0) (at 108.6994 71.12 0)
+      (effects (font (size 1.27 1.27)) (justify left))
+    )
+    (property "Value" "CH340C" (id 1) (at 108.6994 73.66 0)
+      (effects (font (size 1.27 1.27)) (justify left))
+    )
+    (property "Footprint" "Package_SO:SOIC-16_3.9x9.9mm_P1.27mm" (id 2) (at 107.95 69.215 0)
+      (effects (font (size 1.27 1.27)) (justify left) hide)
+    )
+    (property "Datasheet" "https://datasheet.lcsc.com/szlcsc/Jiangsu-Qin-Heng-CH340C_C84681.pdf" (id 3) (at 97.79 34.925 0)
+      (effects (font (size 1.27 1.27)) hide)
+    )
+    (pin "1")
+    (pin "10")
+    (pin "11")
+    (pin "12")
+    (pin "13")
+    (pin "14")
+    (pin "15")
+    (pin "16")
+    (pin "2")
+    (pin "3")
+    (pin "4")
+    (pin "5")
+    (pin "6")
+    (pin "7")
+    (pin "8")
+    (pin "9")
   )
   (sheet_instances
     (path "/" (page "1"))
   )
+  (symbol_instances
+    (path "/0c8083f7-fd19-4041-b9b8-331fd89d43ef"
+      (reference "J1") (unit 1) (value "490107670412") (footprint "Snapeda:490107670412_WURTH_490107670412")
+    )
+    (path "/caf789c1-0df5-453c-b776-75c113270984"
+      (reference "U1") (unit 1) (value "CH340C") (footprint "Package_SO:SOIC-16_3.9x9.9mm_P1.27mm")
+    )
+    (path "/493030e6-a978-4130-8313-802ca2f537b3"
+      (reference "U2") (unit 1) (value "TS3USB30RSWR") (footprint "Snapeda:TS3USB30RSWR_QFN40P140X180X55-10N")
+    )
+    (path "/70d3911e-6489-4c6f-a36c-5e3bbb07c3ef"
+      (reference "U3") (unit 1) (value "CH340C") (footprint "Package_SO:SOIC-16_3.9x9.9mm_P1.27mm")
+    )
+  )
 )
