File: design.kicad_sch (KiCad schematic)
At the start: 4 parts, among them J1 490107670412, U1 CH340C, U2 TS3USB30RSWR, U3 CH340C

Commit message: add components
Parts:
- added J2: TYPE-C-31-M-12, Snapeda:TYPE-C-31-M-12_HRO_TYPE-C-31-M-12, symbol Snapeda:TYPE-C-31-M-12
- added J3: 490107670412, Snapeda:490107670412_WURTH_490107670412, symbol Snapeda:490107670412
- added J4: Conn_02x02_Counter_Clockwise, Connector_PinHeader_2.54mm:PinHeader_2x02_P2.54mm_Vertical, symbol Connector_Generic:Conn_02x02_Counter_Clockwise
- added R1, R2: 5.1k, Resistor_SMD:R_0805_2012Metric, symbol Device:R_Small
- added U4: TS3USB30RSWR, Snapeda:TS3USB30RSWR_QFN40P140X180X55-10N, symbol Snapeda:TS3USB30RSWR
- added U5: TCK108AF,LF, Package_TO_SOT_SMD:SOT-23-5, symbol Power_Management_custom:TCK108AF,LF
Connections:
- net D1+: now reaches U2.1 (D1+)
- net D1+: now also U3.5 (UD+), J4.3 (Pin_3)
- net D2+: now reaches U2.2 (D2+)
- net D2+: now also U1.5 (UD+)
- net D+: now reaches U2.3 (D+)
- net D+: now also J2.A6 (DP1), J2.B6 (DP2), J4.2 (Pin_2)
- net D-: now reaches U2.5 (D-)
- net D-: now also J2.A7 (DN1), J2.B7 (DN2), J4.1 (Pin_1)
- net D2-: now reaches U2.6 (D2-)
- net D2-: now also U1.6 (UD-)
- net D1-: now reaches U2.7 (D1-)
- net D1-: now also U3.6 (UD-), J4.4 (Pin_4)
- net TX2: now reaches U3.2 (TXD)
- net TX2: now also U4.1 (D1+), U4.5 (D-)
- net RX2: now reaches U3.3 (RXD)
- net RX2: now also U4.3 (D+), U4.7 (D1-)
- net TX1: now reaches U1.2 (TXD)
- net TX1: now also U4.2 (D2+)
- net RX1: now reaches U1.3 (RXD)
- net RX1: now also U4.6 (D2-)
- new net: J2.A5 (CC1), R1.2
- new net: J2.B5 (CC2), R2.1
- new net: J2.S1 (SHIELD), J2.S2 (SHIELD), J2.S3 (SHIELD), J2.S4 (SHIELD)
- new net GND: J2.A1_B12 (GND), J2.B1_A12 (GND), R1.1, R2.2
- new net VBUS: J2.A4_B9 (VBUS), J2.B4_A9 (VBUS)
- no-connect marks 0 -> 2
Other:
- note added: "S OE FUNCTION X H Disconnect L L D = D1 H L D = D2"
- note added: "voltage 3v3 5v TX RX switch LED power LED witch switch active Power - reset curcuit"
- moved on the sheet: J1, U1, U2, U3

Commit message: Update design.kicad_sch
Parts:
- added D?: 3.3V, symbol Device:LED_Small
- added D?: VBUS power, symbol Device:LED_Small
- added U?: AP2112K-3.3, Package_TO_SOT_SMD:SOT-23-5, symbol Regulator_Linear:AP2112K-3.3
Changed lines of the file:
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@@
     (pin "1")
+  )
+  (symbol (lib_id "Device:LED_Small") (at 100.965 36.195 0) (mirror y) (unit 1)
+    (in_bom yes) (on_board yes) (fields_autoplaced)
+    (property "Reference" "D?" (id 0) (at 100.9015 29.21 0))
+    (property "Value" "3.3V" (id 1) (at 100.9015 31.75 0))
+    (property "Footprint" "" (id 2) (at 100.965 36.195 90)
+      (effects (font (size 1.27 1.27)) hide)
+    )
+    (property "Datasheet" "~" (id 3) (at 100.965 36.195 90)
+      (effects (font (size 1.27 1.27)) hide)
+    )
+    (pin "1")
+    (pin "2")
   )
   (symbol (lib_id "Snapeda:TS3USB30RSWR") (at 104.14 84.455 0) (mirror y) (unit 1)
@@
     (pin "8")
     (pin "9")
+  )
+  (symbol (lib_id "Device:LED_Small") (at 100.965 24.765 0) (mirror y) (unit 1)
+    (in_bom yes) (on_board yes) (fields_autoplaced)
+    (property "Reference" "D?" (id 0) (at 100.9015 17.78 0))
+    (property "Value" "VBUS power" (id 1) (at 100.9015 20.32 0))
+    (property "Footprint" "" (id 2) (at 100.965 24.765 90)
+      (effects (font (size 1.27 1.27)) hide)
+    )
+    (property "Datasheet" "~" (id 3) (at 100.965 24.765 90)
+      (effects (font (size 1.27 1.27)) hide)
+    )
+    (pin "1")
+    (pin "2")
   )
   (symbol (lib_id "Connector_Generic:Conn_02x02_Counter_Clockwise") (at 105.41 121.285 0) (unit 1)
@@
     (pin "9")
   )
+  (symbol (lib_id "Regulator_Linear:AP2112K-3.3") (at 42.545 31.75 0) (unit 1)
+    (in_bom yes) (on_board yes) (fields_autoplaced)
+    (property "Reference" "U?" (id 0) (at 42.545 21.59 0))
+    (property "Value" "AP2112K-3.3" (id 1) (at 42.545 24.13 0))
+    (property "Footprint" "Package_TO_SOT_SMD:SOT-23-5" (id 2) (at 42.545 23.495 0)
+      (effects (font (size 1.27 1.27)) hide)
+    )
+    (property "Datasheet" "https://www.diodes.com/assets/Datasheets/AP2112.pdf" (id 3) (at 42.545 29.21 0)
+      (effects (font (size 1.27 1.27)) hide)
+    )
+    (pin "1")
+    (pin "2")
+    (pin "3")
+    (pin "4")
+    (pin "5")
+  )
   (symbol (lib_id "Power_Management_custom:TCK108AF,LF") (at 61.595 154.94 0) (unit 1)
     (in_bom yes) (on_board yes) (fields_autoplaced)
@@
       (reference "#PWR0103") (unit 1) (value "GND") (footprint "")
     )
+    (path "/42a72fa9-0b4c-4bca-be32-1db44fee4cf2"
+      (reference "D?") (unit 1) (value "3.3V") (footprint "")
+    )
+    (path "/4c6427e9-1acb-4281-b547-6eb177ad5db2"
+      (reference "D?") (unit 1) (value "VBUS power") (footprint "")
+    )
     (path "/0c8083f7-fd19-4041-b9b8-331fd89d43ef"
       (reference "J1") (unit 1) (value "490107670412") (footprint "Snapeda:490107670412_WURTH_490107670412")
@@
       (reference "U5") (unit 1) (value "TCK108AF,LF") (footprint "Package_TO_SOT_SMD:SOT-23-5")
     )
-  )
+    (path "/765b3629-368a-44c5-9010-d6446b5f3f32"
+      (reference "U?") (unit 1) (value "AP2112K-3.3") (footprint "Package_TO_SOT_SMD:SOT-23-5")
+    )
+  )

Commit message: Update design.kicad_sch
Parts:
- removed J3: 490107670412, Snapeda:490107670412_WURTH_490107670412, symbol Snapeda:490107670412
- removed U1: CH340C, Package_SO:SOIC-16_3.9x9.9mm_P1.27mm, symbol Interface_USB:CH340C
- removed U2: TS3USB30RSWR, Snapeda:TS3USB30RSWR_QFN40P140X180X55-10N, symbol Snapeda:TS3USB30RSWR
- added C? (x2): 1uF, Capacitor_SMD:C_0805_2012Metric, symbol Device:C_Small
- added D?: VDD, symbol Device:LED_Small
- added J?: SKEDD:490107670612, Connector_custom:WURTH_490107670612, symbol Connector_custom:SKEDD{colon}490107670612
- added R? (x2): 0 ohm, symbol Device:R_Small
- added R?: R_Small, symbol Device:R_Small
- added SW?: 5V/3.3V, Button_Switch_SMD:SW_DPDT_CK_JS202011JCQN, symbol Switch:SW_DPDT_x2
- added SW?: EN, Button_Switch_SMD_custom:RKB2, symbol Switch:SW_Push
- added U?: TCK107AF,LF, Package_TO_SOT_SMD:SOT-23-5, symbol Power_Management_custom:TCK107AF,LF
Connections:
- net D+: now also U3.5 (UD+)
- net D-: now also U3.6 (UD-)
- net D1+: no longer U3.5 (UD+)
- net D1-: no longer U3.6 (UD-)
- net GND: now also U?.2 (GND), C?.2, C?.2
- net RX1: now also J1.1, J?.3 (RX/IO9), R?.2; no longer U4.6 (D2-)
- net TX1: now also J?.1 (TX/EN), R?.2; no longer U4.2 (D2+)
- net VBUS: now also U?.1 (VIN), U?.3 (EN), C?.1, SW?.1 (A)
- net UPDI: now reaches J1.4
- net UPDI: now also U4.1 (D1+), J?.6 (D+/UDPI), R?.2
- net +3V3: now reaches U?.5 (VOUT)
- net +3V3: now also C?.1, SW?.3 (C)
- removed net RX2: U3.3 (RXD), U4.3 (D+), U4.7 (D1-)
- removed net TX2: U3.2 (TXD), U4.1 (D1+), U4.5 (D-)
- new net: R?.1, U4.7 (D1-)
- new net: U3.2 (TXD), U4.3 (D+)
- new net: U3.3 (RXD), U4.5 (D-)
- new net RX: R?.1, U4.6 (D2-)
- new net TX: R?.1, U4.2 (D2+)
- new net VDD: SW?.2 (B)
Other:
- moved on the sheet: J1, U3, U4, U5A, U?

Commit message: Update design.kicad_sch
Parts:
- removed U5: TCK108AF,LF, Package_TO_SOT_SMD:SOT-23-5, symbol Power_Management_custom:TCK108AF,LF
- added R?: 5.1k, Resistor_SMD:R_0805_2012Metric, symbol Device:R_Small
- R?: value R_Small -> 1k
Connections:
- net D1+ is gone; now on net RX1: J4.3 (Pin_3)
- net D1- is gone; now on net TX1: J4.4 (Pin_4)
- net UPDI is gone; now on net TX1: J1.4, J?.6 (D+/UDPI), R?.2, U4.1 (D1+)
- net +3V3: now also U3.4 (V3), U4.9 (VCC)
- net D+: no longer J4.2 (Pin_2)
- net D-: no longer J4.1 (Pin_1)
- net GND: now also J1.2, J?.2 (GND), SW?.2, U3.1 (GND), U4.4 (GND), U?.2 (GND)
- net RX: now also J4.2 (Pin_2), U3.3 (RXD), U4.5 (D-); no longer R?.1, U4.6 (D2-)
- net RX1: now also R?.1, U4.7 (D1-); no longer J1.1, J?.3 (RX/IO9)
- net TX: now also J4.1 (Pin_1), U3.2 (TXD), U4.3 (D+); no longer R?.1, U4.2 (D2+)
- net TX1: no longer J?.1 (TX/EN)
- net VDD: now also U3.16 (VCC), U?.5 (VIN), R?.2
- net VCC: now reaches J1.3
- net VCC: now also J?.5 (VIN), U?.1 (VOUT)
- net at U?.3 (Control): now also SW?.1, R?.1
- new net RX2: U4.6 (D2-)
- new net RX_skedd: J1.1, J?.3 (RX/IO9), R?.1
- new net TX2: U4.2 (D2+)
- new net TX_skedd: J?.1 (TX/EN), R?.1
- no-connect marks 2 -> 10
Other:
- moved on the sheet: J4, R?, SW?, U4

Commit message: Update design.kicad_sch
Parts:
- removed D?: VDD, symbol Device:LED_Small
- added D?: VDD, symbol Device:LED_Small
- added R? (x3): 330, Resistor_SMD:R_0805_2012Metric, symbol Device:R_Small
- added SW?: D1/D2, Button_Switch_SMD:SW_DPDT_CK_JS202011JCQN, symbol Switch:SW_DPDT_x2
Connections:
- net +3V3: now also R?.1, SW?.1 (A)
- net GND: now also D?.1 (K), D?.1 (K), U4.8 (~OE), D?.1 (K), SW?.3 (C)
- net VBUS: now also R?.1
- net VDD: now also R?.1
- net at D?.2 (A): now also R?.2 (x2)
- net Switch: now reaches U4.10 (S)
- net Switch: now also SW?.2 (B)
- new net: D?.2 (A), R?.2
Other:
- note removed: "S OE FUNCTION X H Disconnect L L D = D1 H L D = D2"

Commit message: update
Parts:
- removed J?: SKEDD:490107670612, Connector_custom:WURTH_490107670612, symbol Connector_custom:SKEDD{colon}490107670612
- removed R? (x2): 0 ohm, symbol Device:R_Small
- added C3, C4: 0.1uF, Capacitor_SMD:C_0805_2012Metric, symbol Device:C_Small
- D1, D2, D3: renamed from D?; footprint (none) -> LED_SMD:LED_0805_2012Metric
- R6: renamed from R?; footprint (none) -> Resistor_SMD:R_0805_2012Metric
- gave numbers to parts that had none: 11
Connections:
- net RX_skedd is gone; now on net RX1: J1.1
- net +3V3: now also C4.1
- net GND: now also C3.2, C4.2
- net RX: now also J4.4 (Pin_4); no longer J4.2 (Pin_2)
- net TX: now also J4.2 (Pin_2); no longer J4.1 (Pin_1)
- net TX1: now also J4.1 (Pin_1); no longer J4.4 (Pin_4)
- net VDD: now also C3.1
- no-connect marks 10 -> 9

Commit message: update
Parts:
- removed SW1: 5V/3.3V, Button_Switch_SMD:SW_DPDT_CK_JS202011JCQN, symbol Switch:SW_DPDT_x2
- removed SW2: D1/D2, Button_Switch_SMD:SW_DPDT_CK_JS202011JCQN, symbol Switch:SW_DPDT_x2
- added D4: VDD, LED_SMD:LED_0805_2012Metric, symbol Device:LED_Small
- added R7: 330, Resistor_SMD:R_0805_2012Metric, symbol Device:R_Small
- added S1, S2: JS202011JCQN, Snapeda:SW_JS202011JCQN, symbol Snapeda:JS202011JCQN
Connections:
- net +3V3: now also R7.1, S1.3, S2.1
- net GND: now also S1.6, S2.3; no longer D2.1 (K)
- net Switch: now also S2.2
- net VBUS: now also R4.1, S1.1
- net VDD: now also S1.2; no longer R4.1
- new net: D4.2 (A), R7.2
- new net: D2.1 (K), S1.5
- new net: D4.1 (K), S1.7
- no-connect marks 9 -> 12

Commit message: update
Connections:
- net RX: now also J4.2 (Pin_2); no longer J4.4 (Pin_4)
- net RX1: now also J4.1 (Pin_1); no longer J1.1, J4.3 (Pin_3)
- net RX2: now also J1.1
- net TX: now also J4.4 (Pin_4); no longer J4.2 (Pin_2)
- net TX1: now also J4.3 (Pin_3); no longer J4.1 (Pin_1)
- no-connect marks 12 -> 13
Changed lines of the file:
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@@
   (no_connect (at 27.305 91.44))
   (no_connect (at 62.865 83.82))
+  (no_connect (at 62.865 96.52))
   (no_connect (at 96.52 80.645))
   (no_connect (at 116.84 98.425))
@@
     )
   )
-  (global_label "RX1" (shape input) (at 168.91 130.81 0) (fields_autoplaced)
-    (effects (font (size 1.27 1.27)) (justify left))
-    (property "Referenzen zwischen Schaltplänen" "${INTERSHEET_REFS}" (id 0) (at 174.9232 130.8894 0)
-      (effects (font (size 1.27 1.27)) (justify left) hide)
+  (global_label "RX1" (shape input) (at 156.21 128.27 180) (fields_autoplaced)
+    (effects (font (size 1.27 1.27)) (justify right))
+    (property "Referenzen zwischen Schaltplänen" "${INTERSHEET_REFS}" (id 0) (at 150.1968 128.1906 0)
+      (effects (font (size 1.27 1.27)) (justify right) hide)
     )
   )
@@
     )
   )
-  (global_label "RX" (shape input) (at 168.91 128.27 0) (fields_autoplaced)
-    (effects (font (size 1.27 1.27)) (justify left))
-    (property "Referenzen zwischen Schaltplänen" "${INTERSHEET_REFS}" (id 0) (at 173.7137 128.3494 0)
-      (effects (font (size 1.27 1.27)) (justify left) hide)
+  (global_label "RX" (shape input) (at 156.21 130.81 180) (fields_autoplaced)
+    (effects (font (size 1.27 1.27)) (justify right))
+    (property "Referenzen zwischen Schaltplänen" "${INTERSHEET_REFS}" (id 0) (at 151.4063 130.7306 0)
+      (effects (font (size 1.27 1.27)) (justify right) hide)
     )
   )
@@
     )
   )
-  (global_label "TX" (shape input) (at 156.21 130.81 180) (fields_autoplaced)
-    (effects (font (size 1.27 1.27)) (justify right))
-    (property "Referenzen zwischen Schaltplänen" "${INTERSHEET_REFS}" (id 0) (at 151.7087 130.7306 0)
-      (effects (font (size 1.27 1.27)) (justify right) hide)
+  (global_label "TX" (shape input) (at 168.91 128.27 0) (fields_autoplaced)
+    (effects (font (size 1.27 1.27)) (justify left))
+    (property "Referenzen zwischen Schaltplänen" "${INTERSHEET_REFS}" (id 0) (at 173.4113 128.3494 0)
+      (effects (font (size 1.27 1.27)) (justify left) hide)
     )
   )
@@
     )
   )
-  (global_label "RX1" (shape input) (at 231.775 85.09 180) (fields_autoplaced)
+  (global_label "RX2" (shape input) (at 231.775 85.09 180) (fields_autoplaced)
     (effects (font (size 1.27 1.27)) (justify right))
     (property "Referenzen zwischen Schaltplänen" "${INTERSHEET_REFS}" (id 0) (at 225.7618 85.1694 0)
@@
     )
   )
-  (global_label "TX1" (shape input) (at 156.21 128.27 180) (fields_autoplaced)
-    (effects (font (size 1.27 1.27)) (justify right))
-    (property "Referenzen zwischen Schaltplänen" "${INTERSHEET_REFS}" (id 0) (at 150.4991 128.1906 0)
-      (effects (font (size 1.27 1.27)) (justify right) hide)
+  (global_label "TX1" (shape input) (at 168.91 130.81 0) (fields_autoplaced)
+    (effects (font (size 1.27 1.27)) (justify left))
+    (property "Referenzen zwischen Schaltplänen" "${INTERSHEET_REFS}" (id 0) (at 174.6209 130.8894 0)
+      (effects (font (size 1.27 1.27)) (justify left) hide)
     )
   )
