File: design.kicad_sch (KiCad schematic)
At the start: 26 parts, among them J1 490107670412, J2 TYPE-C-31-M-12, J4 Conn_02x02_Counter_Clockwise, SW3 EN, U1 AP2112K-3.3, U2 TCK107AF,LF, U3 CH340C, U4 TS3USB30RSWR

Commit message: update
Parts:
- added TP1, TP2: TestPoint, TestPoint:TestPoint_Pad_D2.0mm, symbol Connector:TestPoint
- D1: value VBUS power -> 5V
- D2: value VDD -> 5V
- D4: value VDD -> 3.3V
- SW3: value EN -> Power cycle
Connections:
- net RX2: now also TP1.1
- net TX2: now also TP2.1

Commit message: cleanup
Parts:
- removed SW3: Power cycle, Button_Switch_SMD_custom:RKB2, symbol Switch:SW_Push
- added S3: Power Cycle, Snapeda:EVP-BFAC1A000_EVPBFAC1A000, symbol Snapeda:EVP-BFAC1A000
- TP1: value TestPoint -> RX2
- TP2: value TestPoint -> TX2
Connections:
- net GND: now also S3.B2 (B')
- net at R9.1, U2.3 (Control): now also S3.B1 (B)
- no-connect marks 13 -> 15
Changed lines of the file:
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@@
   (no_connect (at 116.84 93.345))
   (no_connect (at 27.305 91.44))
+  (no_connect (at 43.815 155.575))
   (no_connect (at 62.865 83.82))
+  (no_connect (at 61.595 155.575))
   (no_connect (at 62.865 96.52))
   (no_connect (at 96.52 80.645))
@@
     (stroke (width 0) (type default) (color 0 0 0 0))
   )
-  (wire (pts (xy 46.355 153.035) (xy 51.435 153.035))
+  (wire (pts (xy 38.735 153.035) (xy 43.815 153.035))
     (stroke (width 0) (type default) (color 0 0 0 0))
   )
@@
     (pin "1")
   )
+  (symbol (lib_id "Snapeda:EVP-BFAC1A000") (at 48.895 150.495 0) (unit 1)
+    (in_bom yes) (on_board yes) (fields_autoplaced)
+    (property "Reference" "S3" (id 0) (at 52.705 144.78 0))
+    (property "Value" "Power Cycle" (id 1) (at 52.705 147.32 0))
+    (property "Footprint" "Snapeda:EVP-BFAC1A000_EVPBFAC1A000" (id 2) (at 48.895 150.495 0)
+      (effects (font (size 1.27 1.27)) (justify bottom) hide)
+    )
+    (property "Datasheet" "" (id 3) (at 48.895 150.495 0)
+      (effects (font (size 1.27 1.27)) hide)
+    )
+    (property "MANUFACTURER_NAME" "Panasonic" (id 4) (at 48.895 150.495 0)
+      (effects (font (size 1.27 1.27)) (justify bottom) hide)
+    )
+    (property "MF" "Panasonic Electronic" (id 5) (at 48.895 150.495 0)
+      (effects (font (size 1.27 1.27)) (justify bottom) hide)
+    )
+    (property "MOUSER_PRICE-STOCK" "https://www.mouser.com/Search/Refine.aspx?Keyword=667-EVP-BFAC1A000" (id 6) (at 48.895 150.495 0)
+      (effects (font (size 1.27 1.27)) (justify bottom) hide)
+    )
+    (property "DESCRIPTION" "Tactile Switches 6.0x6.0x3.4mm 2N w/4 Term .25mm Trvl IP67" (id 7) (at 48.895 150.495 0)
+      (effects (font (size 1.27 1.27)) (justify bottom) hide)
+    )
+    (property "ALLIED_NUMBER" "70900260" (id 8) (at 48.895 150.495 0)
+      (effects (font (size 1.27 1.27)) (justify bottom) hide)
+    )
+    (property "RS_PART_NUMBER" "" (id 9) (at 48.895 150.495 0)
+      (effects (font (size 1.27 1.27)) (justify bottom) hide)
+    )
+    (property "ALLIED_PRICE-STOCK" "https://www.alliedelec.com/panasonic-evp-bfac1a000/70900260/" (id 10) (at 48.895 150.495 0)
+      (effects (font (size 1.27 1.27)) (justify bottom) hide)
+    )
+    (property "Price" "None" (id 11) (at 48.895 150.495 0)
+      (effects (font (size 1.27 1.27)) (justify bottom) hide)
+    )
+    (property "MOUSER_PART_NUMBER" "667-EVP-BFAC1A000" (id 12) (at 48.895 150.495 0)
+      (effects (font (size 1.27 1.27)) (justify bottom) hide)
+    )
+    (property "Check_prices" "https://www.snapeda.com/parts/EVP-BFAC1A000/Panasonic+Electronic+Components/view-part/?ref=eda" (id 13) (at 48.895 150.495 0)
+      (effects (font (size 1.27 1.27)) (justify bottom) hide)
+    )
+    (property "HEIGHT" "3.7mm" (id 14) (at 48.895 150.495 0)
+      (effects (font (size 1.27 1.27)) (justify bottom) hide)
+    )
+    (property "SnapEDA_Link" "https://www.snapeda.com/parts/EVP-BFAC1A000/Panasonic+Electronic+Components/view-part/?ref=snap" (id 15) (at 48.895 150.495 0)
+      (effects (font (size 1.27 1.27)) (justify bottom) hide)
+    )
+    (property "MP" "EVP-BFAC1A000" (id 16) (at 48.895 150.495 0)
+      (effects (font (size 1.27 1.27)) (justify bottom) hide)
+    )
+    (property "Package" "None" (id 17) (at 48.895 150.495 0)
+      (effects (font (size 1.27 1.27)) (justify bottom) hide)
+    )
+    (property "Purchase-URL" "https://www.snapeda.com/api/url_track_click_mouser/?unipart_id=565679&manufacturer=Panasonic Electronic&part_name=EVP-BFAC1A000&search_term=evp-bfac1a000" (id 18) (at 48.895 150.495 0)
+      (effects (font (size 1.27 1.27)) (justify bottom) hide)
+    )
+    (property "RS_PRICE-STOCK" "" (id 19) (at 48.895 150.495 0)
+      (effects (font (size 1.27 1.27)) (justify bottom) hide)
+    )
+    (property "Description" "\nPanasonic 0.25mm travel with 4 Terminal | Panasonic Electronic Components EVP-BFAC1A000\n" (id 20) (at 48.895 150.495 0)
+      (effects (font (size 1.27 1.27)) (justify bottom) hide)
+    )
+    (property "Availability" "In Stock" (id 21) (at 48.895 150.495 0)
+      (effects (font (size 1.27 1.27)) (justify bottom) hide)
+    )
+    (property "MANUFACTURER_PART_NUMBER" "EVP-BFAC1A000" (id 22) (at 48.895 150.495 0)
+      (effects (font (size 1.27 1.27)) (justify bottom) hide)
+    )
+    (pin "A1")
+    (pin "A2")
+    (pin "B1")
+    (pin "B2")
+  )
   (symbol (lib_id "power:+3V3") (at 193.675 61.595 0) (unit 1)
     (in_bom yes) (on_board yes) (fields_autoplaced)
@@
       (effects (font (size 1.27 1.27)) (justify left))
     )
-    (property "Value" "TestPoint" (id 1) (at 223.52 128.1429 0)
+    (property "Value" "RX2" (id 1) (at 223.52 128.1429 0)
       (effects (font (size 1.27 1.27)) (justify left))
     )
@@
       (effects (font (size 1.27 1.27)) (justify left))
     )
-    (property "Value" "TestPoint" (id 1) (at 238.76 128.1429 0)
+    (property "Value" "TX2" (id 1) (at 238.76 128.1429 0)
       (effects (font (size 1.27 1.27)) (justify left))
     )
@@
     (pin "1")
   )
-  (symbol (lib_id "Switch:SW_Push") (at 56.515 153.035 0) (mirror y) (unit 1)
-    (in_bom yes) (on_board yes) (fields_autoplaced)
-    (property "Reference" "SW3" (id 0) (at 56.515 145.415 0))
-    (property "Value" "Power cycle" (id 1) (at 56.515 147.955 0))
-    (property "Footprint" "Button_Switch_SMD_custom:RKB2" (id 2) (at 56.515 147.955 0)
-      (effects (font (size 1.27 1.27)) hide)
-    )
-    (property "Datasheet" "~" (id 3) (at 56.515 147.955 0)
-      (effects (font (size 1.27 1.27)) hide)
-    )
-    (pin "1")
-    (pin "2")
-  )
   (symbol (lib_id "power:VDD") (at 106.68 73.025 0) (mirror y) (unit 1)
     (in_bom yes) (on_board yes)
@@
     (pin "2")
   )
-  (symbol (lib_id "power:GND") (at 46.355 153.035 0) (unit 1)
+  (symbol (lib_id "power:GND") (at 38.735 153.035 0) (unit 1)
     (in_bom yes) (on_board yes) (fields_autoplaced)
-    (property "Reference" "#PWR0117" (id 0) (at 46.355 159.385 0)
+    (property "Reference" "#PWR0117" (id 0) (at 38.735 159.385 0)
       (effects (font (size 1.27 1.27)) hide)
     )
-    (property "Value" "GND" (id 1) (at 46.355 158.115 0))
-    (property "Footprint" "" (id 2) (at 46.355 153.035 0)
+    (property "Value" "GND" (id 1) (at 38.735 158.115 0))
+    (property "Footprint" "" (id 2) (at 38.735 153.035 0)
       (effects (font (size 1.27 1.27)) hide)
     )
-    (property "Datasheet" "" (id 3) (at 46.355 153.035 0)
+    (property "Datasheet" "" (id 3) (at 38.735 153.035 0)
       (effects (font (size 1.27 1.27)) hide)
     )
@@
       (reference "S2") (unit 1) (value "JS202011JCQN") (footprint "Snapeda:SW_JS202011JCQN")
     )
-    (path "/c416f21f-6180-4d2c-aa6b-aedf8166fa57"
-      (reference "SW3") (unit 1) (value "Power cycle") (footprint "Button_Switch_SMD_custom:RKB2")
+    (path "/65978a9e-5e10-431c-ada0-ed1a7f686d25"
+      (reference "S3") (unit 1) (value "Power Cycle") (footprint "Snapeda:EVP-BFAC1A000_EVPBFAC1A000")
     )
     (path "/95cb8cc0-b0b1-4ef0-8ea6-07632f0b0aca"
-      (reference "TP1") (unit 1) (value "TestPoint") (footprint "TestPoint:TestPoint_Pad_D2.0mm")
+      (reference "TP1") (unit 1) (value "RX2") (footprint "TestPoint:TestPoint_Pad_D2.0mm")
     )
     (path "/a3cc14d5-da5a-4b67-a7cc-febefd92fe93"
-      (reference "TP2") (unit 1) (value "TestPoint") (footprint "TestPoint:TestPoint_Pad_D2.0mm")
+      (reference "TP2") (unit 1) (value "TX2") (footprint "TestPoint:TestPoint_Pad_D2.0mm")
     )
     (path "/765b3629-368a-44c5-9010-d6446b5f3f32"

Commit message: small changes
Parts:
- added TP3: 3.3V, TestPoint:TestPoint_Pad_D2.0mm, symbol Connector:TestPoint
- added TP4: 5V, TestPoint:TestPoint_Pad_D2.0mm, symbol Connector:TestPoint
- added TP5: VCC, TestPoint:TestPoint_Pad_D2.0mm, symbol Connector:TestPoint
- added TP? (x2): GND, TestPoint:TestPoint_Pad_D2.0mm, symbol Connector:TestPoint
Connections:
- net +3V3: now also TP3.1
- net GND: now also TP?.1, TP?.1
- net VBUS: now also TP4.1
- net VCC: now also TP5.1
Other:
- moved on the sheet: TP1, TP2

Commit message: update
Parts:
- gave numbers to parts that had none: 2
Changed lines of the file:
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@@
   (symbol (lib_id "power:GND") (at 221.615 134.62 0) (unit 1)
     (in_bom yes) (on_board yes) (fields_autoplaced)
-    (property "Reference" "#PWR?" (id 0) (at 221.615 140.97 0)
+    (property "Reference" "#PWR0139" (id 0) (at 221.615 140.97 0)
       (effects (font (size 1.27 1.27)) hide)
     )
@@
   (symbol (lib_id "power:GND") (at 212.09 134.62 0) (unit 1)
     (in_bom yes) (on_board yes) (fields_autoplaced)
-    (property "Reference" "#PWR?" (id 0) (at 212.09 140.97 0)
+    (property "Reference" "#PWR0138" (id 0) (at 212.09 140.97 0)
       (effects (font (size 1.27 1.27)) hide)
     )
@@
   (symbol (lib_id "Connector:TestPoint") (at 212.09 130.175 0) (unit 1)
     (in_bom yes) (on_board yes) (fields_autoplaced)
-    (property "Reference" "TP?" (id 0) (at 213.995 125.6029 0)
+    (property "Reference" "TP6" (id 0) (at 213.995 125.6029 0)
       (effects (font (size 1.27 1.27)) (justify left))
     )
@@
   (symbol (lib_id "Connector:TestPoint") (at 221.615 130.175 0) (unit 1)
     (in_bom yes) (on_board yes) (fields_autoplaced)
-    (property "Reference" "TP?" (id 0) (at 223.52 125.6029 0)
+    (property "Reference" "TP7" (id 0) (at 223.52 125.6029 0)
       (effects (font (size 1.27 1.27)) (justify left))
     )
@@
       (reference "#PWR0137") (unit 1) (value "VCC") (footprint "")
     )
+    (path "/2f0ea48a-577c-40ab-86ef-e29840bd6f74"
+      (reference "#PWR0138") (unit 1) (value "GND") (footprint "")
+    )
     (path "/22b3a896-2430-494e-927f-3a3865d8dac2"
-      (reference "#PWR?") (unit 1) (value "GND") (footprint "")
-    )
-    (path "/2f0ea48a-577c-40ab-86ef-e29840bd6f74"
-      (reference "#PWR?") (unit 1) (value "GND") (footprint "")
+      (reference "#PWR0139") (unit 1) (value "GND") (footprint "")
     )
     (path "/8ff5159f-9d2d-4c22-b93a-c6c716137c33"
@@
     )
     (path "/62ebb2e8-9966-4d25-8279-84394c505879"
-      (reference "TP?") (unit 1) (value "GND") (footprint "TestPoint:TestPoint_Pad_D2.0mm")
+      (reference "TP6") (unit 1) (value "GND") (footprint "TestPoint:TestPoint_Pad_D2.0mm")
     )
     (path "/cba6d5c0-5de0-4bc6-a0fc-894d369b41b2"
-      (reference "TP?") (unit 1) (value "GND") (footprint "TestPoint:TestPoint_Pad_D2.0mm")
+      (reference "TP7") (unit 1) (value "GND") (footprint "TestPoint:TestPoint_Pad_D2.0mm")
     )
     (path "/765b3629-368a-44c5-9010-d6446b5f3f32"

Commit message: update for logo
Parts:
- added logo: VCC, TestPoint:TestPoint_Pad_D2.0mm, symbol Connector:TestPoint
Connections:
- no-connect marks 15 -> 16
Changed lines of the file:
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@@
   (no_connect (at 43.815 155.575))
   (no_connect (at 62.865 83.82))
+  (no_connect (at 266.7 154.305))
   (no_connect (at 61.595 155.575))
   (no_connect (at 62.865 96.52))
@@
     (pin "1")
   )
+  (symbol (lib_id "Connector:TestPoint") (at 266.7 154.305 0) (unit 1)
+    (in_bom yes) (on_board yes) (fields_autoplaced)
+    (property "Reference" "logo" (id 0) (at 269.24 149.7329 0)
+      (effects (font (size 1.27 1.27)) (justify left))
+    )
+    (property "Value" "VCC" (id 1) (at 269.24 152.2729 0)
+      (effects (font (size 1.27 1.27)) (justify left))
+    )
+    (property "Footprint" "TestPoint:TestPoint_Pad_D2.0mm" (id 2) (at 271.78 154.305 0)
+      (effects (font (size 1.27 1.27)) hide)
+    )
+    (property "Datasheet" "~" (id 3) (at 271.78 154.305 0)
+      (effects (font (size 1.27 1.27)) hide)
+    )
+    (pin "1")
+  )
   (symbol (lib_id "Device:LED_Small") (at 177.8 26.162 0) (mirror x) (unit 1)
     (in_bom yes) (on_board yes) (fields_autoplaced)
@@
       (reference "U4") (unit 1) (value "TS3USB30RSWR") (footprint "Snapeda:TS3USB30RSWR_QFN40P140X180X55-10N")
     )
+    (path "/30cad120-e725-449e-a695-7e737ec28185"
+      (reference "logo") (unit 1) (value "VCC") (footprint "TestPoint:TestPoint_Pad_D2.0mm")
+    )
   )

Commit message: remove logo
Parts:
- removed logo: VCC, TestPoint:TestPoint_Pad_D2.0mm, symbol Connector:TestPoint
Connections:
- no-connect marks 16 -> 15
Changed lines of the file:
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@@
   (no_connect (at 43.815 155.575))
   (no_connect (at 62.865 83.82))
-  (no_connect (at 266.7 154.305))
   (no_connect (at 61.595 155.575))
   (no_connect (at 62.865 96.52))
@@
     (pin "1")
   )
-  (symbol (lib_id "Connector:TestPoint") (at 266.7 154.305 0) (unit 1)
-    (in_bom yes) (on_board yes) (fields_autoplaced)
-    (property "Reference" "logo" (id 0) (at 269.24 149.7329 0)
-      (effects (font (size 1.27 1.27)) (justify left))
-    )
-    (property "Value" "VCC" (id 1) (at 269.24 152.2729 0)
-      (effects (font (size 1.27 1.27)) (justify left))
-    )
-    (property "Footprint" "TestPoint:TestPoint_Pad_D2.0mm" (id 2) (at 271.78 154.305 0)
-      (effects (font (size 1.27 1.27)) hide)
-    )
-    (property "Datasheet" "~" (id 3) (at 271.78 154.305 0)
-      (effects (font (size 1.27 1.27)) hide)
-    )
-    (pin "1")
-  )
   (symbol (lib_id "Device:LED_Small") (at 177.8 26.162 0) (mirror x) (unit 1)
     (in_bom yes) (on_board yes) (fields_autoplaced)
@@
       (reference "U4") (unit 1) (value "TS3USB30RSWR") (footprint "Snapeda:TS3USB30RSWR_QFN40P140X180X55-10N")
     )
-    (path "/30cad120-e725-449e-a695-7e737ec28185"
-      (reference "logo") (unit 1) (value "VCC") (footprint "TestPoint:TestPoint_Pad_D2.0mm")
-    )
   )
