File: design.kicad_pcb (KiCad board)
At the start: 2 copper layers, 81.5 x 51 mm, 4 parts, among them J1 490107670412, U1 CH340C, U2 TS3USB30RSWR, U3 CH340C

Commit message: add components
Parts:
- added J2: TYPE-C-31-M-12, Snapeda:TYPE-C-31-M-12_HRO_TYPE-C-31-M-12, F.Cu at (162.2, 98.7)
- added J3: 490107670412, Snapeda:490107670412_WURTH_490107670412, F.Cu at (178.5, 107.0)
- added J4: Conn_02x02_Counter_Clockwise, Connector_PinHeader_2.54mm:PinHeader_2x02_P2.54mm_Vertical, F.Cu at (143.5, 101.5)
- added R1: 5.1k, Resistor_SMD:R_0805_2012Metric, F.Cu at (150.6, 103.6)
- added R2: 5.1k, Resistor_SMD:R_0805_2012Metric, F.Cu at (150.6, 100.7)
- added U4: TS3USB30RSWR, Snapeda:TS3USB30RSWR_QFN40P140X180X55-10N, F.Cu at (172.6, 92.0)
- added U5: TCK108AF,LF, Package_TO_SOT_SMD:SOT-23-5, F.Cu at (174.0, 112.8)
Connections:
- U1 pad 2: unconnected-(U1-Pad2) -> TX1
- U1 pad 3: unconnected-(U1-Pad3) -> RX1
- U1 pad 5: unconnected-(U1-Pad5) -> D2+
- U1 pad 6: unconnected-(U1-Pad6) -> D2-
- U2 pad 1: unconnected-(U2-Pad1) -> D1+
- U2 pad 2: unconnected-(U2-Pad2) -> D2+
- U2 pad 3: unconnected-(U2-Pad3) -> D+
- U2 pad 5: unconnected-(U2-Pad5) -> D-
- U2 pad 6: unconnected-(U2-Pad6) -> D2-
- U2 pad 7: unconnected-(U2-Pad7) -> D1-
- U3 pad 2: unconnected-(U3-Pad2) -> TX2
- U3 pad 3: unconnected-(U3-Pad3) -> RX2
- U3 pad 5: unconnected-(U3-Pad5) -> D1+
- U3 pad 6: unconnected-(U3-Pad6) -> D1-

Commit message: update
Parts:
- removed J3: 490107670412, Snapeda:490107670412_WURTH_490107670412
- removed U5: TCK108AF,LF, Package_TO_SOT_SMD:SOT-23-5
- added C1: 1uF, Capacitor_SMD:C_0805_2012Metric, F.Cu at (129.0, 73.8)
- added C2: 1uF, Capacitor_SMD:C_0805_2012Metric, F.Cu at (133.2, 76.1)
- added C3: 0.1uF, Capacitor_SMD:C_0805_2012Metric, F.Cu at (141.0, 87.0)
- added C4: 0.1uF, Capacitor_SMD:C_0805_2012Metric, F.Cu at (153.5, 95.0)
- added D1: VBUS power, LED_SMD:LED_0805_2012Metric, F.Cu at (155.2, 71.5)
- added D2: VDD, LED_SMD:LED_0805_2012Metric, F.Cu at (145.5, 71.5)
- added D3: 3.3V, LED_SMD:LED_0805_2012Metric, F.Cu at (150.5, 71.5)
- added R3: 330, Resistor_SMD:R_0805_2012Metric, F.Cu at (155.0, 76.5)
- added R4: 330, Resistor_SMD:R_0805_2012Metric, F.Cu at (145.5, 76.5)
- added R5: 330, Resistor_SMD:R_0805_2012Metric, F.Cu at (150.5, 76.5)
- added R6: 1k, Resistor_SMD:R_0805_2012Metric, F.Cu at (156.0, 95.0)
- added R9: 5.1k, Resistor_SMD:R_0805_2012Metric, F.Cu at (172.8, 84.0)
- added SW1: 5V/3.3V, Button_Switch_SMD:SW_DPDT_CK_JS202011JCQN, F.Cu at (129.8, 82.5)
- added SW2: D1/D2, Button_Switch_SMD:SW_DPDT_CK_JS202011JCQN, F.Cu at (150.0, 82.5)
- added SW3: EN, Button_Switch_SMD_custom:RKB2, F.Cu at (166.8, 84.0)
- U1: value CH340C -> AP2112K-3.3; footprint Package_SO:SOIC-16_3.9x9.9mm_P1.27mm -> Package_TO_SOT_SMD:SOT-23-5
- U2: value TS3USB30RSWR -> TCK107AF,LF; footprint Snapeda:TS3USB30RSWR_QFN40P140X180X55-10N -> Package_TO_SOT_SMD:SOT-23-5
- moved J2 43.4 mm to (119.0, 94.6), turned to -90 degrees
- moved R1 32.5 mm to (122.0, 88.1), turned to 180 degrees
- moved R2 28.6 mm to (122.0, 101.1)
- moved U1 25.0 mm to (130.0, 76.5)
- moved U4 23.3 mm to (149.5, 95.0), turned to -90 degrees
- moved J4 20.0 mm to (162.8, 96.3), turned to 180 degrees
- moved J1 14.3 mm to (172.5, 94.0), turned to 90 degrees
- moved U3 4.76 mm to (141.0, 94.5)
- moved U2 3.50 mm to (160.0, 84.0), turned to 180 degrees
Connections:
- J1 pad 1: unconnected-(J1-Pad1) -> RX1
- J1 pad 2: unconnected-(J1-Pad2) -> GND
- J1 pad 3: unconnected-(J1-Pad3) -> VCC
- J1 pad 4: unconnected-(J1-Pad4) -> TX1
- J4 pad 1: D- -> TX1
- J4 pad 2: D+ -> TX
- J4 pad 3: D1+ -> RX1
- J4 pad 4: D1- -> RX
- U1 pad 1: unconnected-(U1-Pad1) -> VBUS
- U1 pad 2: TX1 -> GND
- U1 pad 3: RX1 -> VBUS
- U1 pad 5: D2+ -> +3V3
- U2 pad 1: D1+ -> VCC
- U2 pad 2: D2+ -> GND
- U2 pad 3: D+ -> Net-(R9-Pad1)
- U2 pad 5: D- -> VDD
- U3 pad 1: unconnected-(U3-Pad1) -> GND
- U3 pad 16: unconnected-(U3-Pad16) -> VDD
- U3 pad 2: TX2 -> TX
- U3 pad 3: RX2 -> RX
- U3 pad 4: unconnected-(U3-Pad4) -> +3V3
- U3 pad 5: D1+ -> D+
- U3 pad 6: D1- -> D-
- U4 pad 1: TX2 -> TX1
- U4 pad 10: unconnected-(U4-Pad10) -> Switch
- U4 pad 2: TX1 -> TX2
- U4 pad 3: RX2 -> TX
- U4 pad 4: unconnected-(U4-Pad4) -> GND
- U4 pad 5: TX2 -> RX
- U4 pad 6: RX1 -> RX2
- U4 pad 7: RX2 -> RX1
- U4 pad 8: unconnected-(U4-Pad8) -> GND
- U4 pad 9: unconnected-(U4-Pad9) -> +3V3
Routing:
- net D-: track 0.00 -> 23.5 mm, vias 0 -> 2
- net D+: track 0.00 -> 21.7 mm
- net Net-(J2-PadA5): track 0.00 -> 7.00 mm
- net Net-(J2-PadB5): track 0.00 -> 6.31 mm
- net VDD: track 0.00 -> 4.68 mm
- net +3V3: track 0.00 -> 3.53 mm
- net (no net): vias 1 -> 0
- added copper zone on F.Cu, net VBUS
Other:
- board text removed: "sdfs dkajölskdj"

Commit message: update
Parts:
- removed SW1: 5V/3.3V, Button_Switch_SMD:SW_DPDT_CK_JS202011JCQN
- removed SW2: D1/D2, Button_Switch_SMD:SW_DPDT_CK_JS202011JCQN
- added D4: VDD, LED_SMD:LED_0805_2012Metric, F.Cu at (164.0, 79.0)
- added R7: 330, Resistor_SMD:R_0805_2012Metric, F.Cu at (168.4, 79.0)
- added S1: JS202011JCQN, Snapeda:SW_JS202011JCQN, F.Cu at (146.8, 78.5)
- added S2: JS202011JCQN, Snapeda:SW_JS202011JCQN, F.Cu at (152.7, 78.5)
- moved D1 29.3 mm to (157.0, 100.8)
- moved D2 29.3 mm to (147.3, 100.8)
- moved D3 29.3 mm to (152.3, 100.8)
- moved R3 27.8 mm to (156.8, 104.2)
- moved R4 27.8 mm to (147.3, 104.2)
- moved R5 27.8 mm to (152.3, 104.2)
- moved SW3 21.3 mm to (148.5, 95.0), turned to 90 degrees
- moved C1 13.9 mm to (129.2, 87.6)
- moved C2 13.9 mm to (133.5, 90.0)
- moved U1 13.9 mm to (130.2, 90.4)
- moved R9 11.0 mm to (162.5, 88.0)
- moved U2 4.37 mm to (158.2, 88.0)
- moved U4 4.00 mm to (153.5, 95.0)
- moved J4 3.25 mm to (166.0, 96.3)
- moved C4 3.00 mm to (156.5, 95.0)
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Connections:
- D2 pad 1: GND -> Net-(D2-Pad1)
- R4 pad 1: VDD -> VBUS
Routing:
- net +3V3: track 3.53 -> 0.00 mm
- removed copper zone on F.Cu, net VBUS

Commit message: update
Parts:
- added REF**: TestPoint_Pad_D2.0mm, TestPoint:TestPoint_Pad_D2.0mm, B.Cu at (164.5, 88.5)
- added REF**: TestPoint_Pad_D2.0mm, TestPoint:TestPoint_Pad_D2.0mm, B.Cu at (164.5, 100.2)
- moved R7 40.1 mm to (137.9, 105.0), turned to 180 degrees
- moved D4 39.7 mm to (134.0, 105.0)
- moved R3 37.0 mm to (125.2, 85.0)
- moved D1 32.0 mm to (129.2, 85.0), turned to 180 degrees
- moved R5 27.1 mm to (133.2, 85.0)
- moved S1 26.7 mm to (131.0, 100.0), turned to 90 degrees
- moved D3 21.8 mm to (137.2, 85.0), turned to 180 degrees
- moved D2 21.7 mm to (126.0, 105.0)
- moved R4 17.3 mm to (130.0, 105.0), turned to 180 degrees
- moved R9 16.8 mm to (153.2, 102.0)
- moved U2 14.0 mm to (157.8, 102.0)
- moved S2 9.70 mm to (150.8, 88.0), turned to 90 degrees
- moved C3 0.75 mm to (141.0, 87.8)
- moved J1 0.75 mm to (173.2, 94.8)
- moved C1 0.36 mm to (129.2, 87.2)
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Connections:
- J1 pad 1: RX1 -> RX2
- J2 pad S1: Net-(J2-PadS1) -> unconnected-(J2-PadS1)
- J2 pad S2: Net-(J2-PadS1) -> unconnected-(J2-PadS1)
- J2 pad S3: Net-(J2-PadS1) -> unconnected-(J2-PadS1)
- J2 pad S4: Net-(J2-PadS1) -> unconnected-(J2-PadS1)
- J4 pad 1: TX1 -> RX1
- J4 pad 2: TX -> RX
- J4 pad 3: RX1 -> TX1
- J4 pad 4: RX -> TX
Routing:
- net +3V3: track 0.00 -> 67.4 mm, vias 0 -> 4
- net VDD: track 4.68 -> 56.1 mm, vias 0 -> 2
- net VBUS: track 0.00 -> 37.0 mm, vias 0 -> 2
- net RX: track 0.00 -> 29.4 mm
- net TX: track 0.00 -> 28.7 mm
- net TX1: track 0.00 -> 25.0 mm
- net RX2: track 0.00 -> 24.3 mm, vias 0 -> 1
- net VCC: track 0.00 -> 18.2 mm
- net Net-(R9-Pad1): track 0.00 -> 15.2 mm
- net RX1: track 0.00 -> 15.1 mm, vias 0 -> 1
- net TX2: track 0.00 -> 13.9 mm, vias 0 -> 1
- net GND: track 0.05 -> 10.8 mm, vias 0 -> 8
- net Switch: track 0.00 -> 8.31 mm, vias 0 -> 2
- net Net-(D2-Pad1): track 0.00 -> 8.24 mm, vias 0 -> 2
- net Net-(D4-Pad1): track 0.00 -> 7.08 mm, vias 0 -> 2
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- added copper zone on B.Cu, net GND
- added copper zone on F.Cu, net GND

Commit message: update
Parts:
- removed REF** (x2): TestPoint_Pad_D2.0mm, TestPoint:TestPoint_Pad_D2.0mm
- added TP1: RX2, TestPoint:TestPoint_Pad_D2.0mm, B.Cu at (164.2, 100.2)
- added TP2: TX2, TestPoint:TestPoint_Pad_D2.0mm, B.Cu at (164.2, 88.8)
- D1: value VBUS power -> 5V
- D2: value VDD -> 5V
- D4: value VDD -> 3.3V
- SW3: value EN -> Power cycle
Routing:
- net Net-(R9-Pad1): track 15.2 -> 21.9 mm, vias 0 -> 2
- net GND: track 10.8 -> 14.1 mm, vias 8 -> 9
Other:
- board text added: "D1"
- board text added: "D2"
- board text added: "Power Rail"
- board text added: "Selected Volatge"

Commit message: cleanup
Parts:
- removed SW3: Power cycle, Button_Switch_SMD_custom:RKB2
- added S3: Power Cycle, Snapeda:EVP-BFAC1A000_EVPBFAC1A000, F.Cu at (148.2, 94.9)
Routing:
- net Net-(R9-Pad1): track 21.9 -> 12.3 mm, vias 2 -> 0
- net +3V3: track 67.4 -> 66.6 mm
Other:
- board size 81.5 x 51 mm -> 61.2 x 35.8 mm
- board text added: "GND"
- board text added: "TR_MCU"
- board text added: "TX_MCU"
- board text added: "UPDI"
- board text added: "VCC"
- board text removed: "D1"
- board text removed: "D2"

Commit message: small changes
Parts:
- added REF**: KiCad-Logo2_5mm_SilkScreen, Symbol:KiCad-Logo2_5mm_SilkScreen, B.Cu at (131.5, 82.2)
- added TP3: 3.3V, TestPoint:TestPoint_Pad_D2.0mm, F.Cu at (161.2, 82.5)
- added TP4: 5V, TestPoint:TestPoint_Pad_D2.0mm, F.Cu at (120.8, 108.2)
- added TP5: VCC, TestPoint:TestPoint_Pad_D2.0mm, F.Cu at (171.8, 108.2)
- added TP6: GND, TestPoint:TestPoint_Pad_D2.0mm, F.Cu at (154.0, 108.2)
- added TP7: GND, TestPoint:TestPoint_Pad_D2.0mm, F.Cu at (169.8, 82.5)
Routing:
- net +3V3: track 66.6 -> 83.4 mm
- net VBUS: track 37.0 -> 48.2 mm
- net VCC: track 18.2 -> 25.7 mm
Other:
- board text added: "RX-RX1"
- board text added: "TX-TX1"

Commit message: update
Parts:
- renumbered REF** to ?
Changed lines of the file:
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@@
     (tags "Logo KiCad")
     (attr exclude_from_pos_files exclude_from_bom)
-    (fp_text reference "REF**" (at 0 5.08) (layer "B.SilkS") hide
+    (fp_text reference "" (at 0 5.08) (layer "B.SilkS") hide
       (effects (font (size 1 1) (thickness 0.15)) (justify mirror))
     )
