File: design.kicad_pcb (KiCad board)
At the start: 2 copper layers, 61.2 x 35.8 mm, 34 parts, among them J1 490107670412, J2 TYPE-C-31-M-12, J4 Conn_02x02_Counter_Clockwise, U1 AP2112K-3.3, U2 TCK107AF,LF, U3 CH340C, U4 TS3USB30RSWR

Commit message: update for logo
Parts:
- gave numbers to parts that had none: 1
Changed lines of the file:
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@@
     (tags "Logo KiCad")
     (attr exclude_from_pos_files exclude_from_bom)
-    (fp_text reference "" (at 0 5.08) (layer "B.SilkS") hide
+    (fp_text reference "logo" (at 0 5.08) (layer "B.SilkS") hide
       (effects (font (size 1 1) (thickness 0.15)) (justify mirror))
     )

Commit message: remove logo
Parts:
- removed logo: KiCad-Logo2_5mm_SilkScreen, Symbol:KiCad-Logo2_5mm_SilkScreen
